File: TP PP HRC VEHICULO/TP PP HRC VEHICULO.kicad_pcb (KiCad board)
At the start: 2 copper layers, 100 x 100 mm, 56 parts, among them J1 Screw_Terminal_01x02, J10 Conn_01x04_Pin, J11 Screw_Terminal_01x02, J2 Conn_01x01_Pin, J3 Conn_01x01_Pin, J4 Screw_Terminal_01x03, J5 Screw_Terminal_01x03, J6 Conn_01x04_Pin, J7 USB_B, J8 Conn_01x02_Pin, J9 Conn_01x04_Pin, K1 Relay_SPDT, K2 Relay_SPDT, Q1 S8050, Q2 S8050, Q3 S8050, SW1 SW_Push, SW2 SW_Push, SW3 SW_DPST_x2, U1 ESP32-Devkit-V1, U2 LM317L_TO92, U3 LM317L_TO92

Commit message: placa actualizada
Parts:
- D5: value LED -> LEDrele1
- D6: value LED -> led_rele2
- moved Drele12 181.6 mm to (179.8, 66.3)
- moved Drele1 175.7 mm to (180.8, 71.9)
- moved borrele1 167.2 mm to (201.2, 100.8), turned to 180 degrees
- moved SWusb1 143.6 mm to (211.8, 136.7), turned to 180 degrees
- moved bornrele2 143.4 mm to (182.9, 127.5), turned to 90 degrees
- moved SW1 121.7 mm to (167.1, 68.6), turned to 90 degrees
- moved J5vgnd1 95.0 mm to (167.1, 137.7), turned to -90 degrees
- moved SW2 84.4 mm to (126.2, 84.6)
- moved Ruv21 83.5 mm to (119.4, 154.2)
- moved Rldr2 76.2 mm to (147.6, 120.9)
- moved Cuv21 74.2 mm to (137.4, 159.8), turned to 180 degrees
- moved K1 72.8 mm to (192.8, 86.4), turned to 0 degrees
- moved K2 72.7 mm to (206.9, 121.9), turned to 180 degrees
- moved Uv2 71.1 mm to (136.7, 152.7), turned to -90 degrees
- moved Ruv2 70.5 mm to (144.3, 160.0)
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- renumbered C4 to CUv2, C2 to Cu1, C3 to Cu2, C1 to Cu3, C5 to Cuv21, C6 to Cuv22, D7 to Drele1, D8 to Drele12, D9 to Dusb1, J1 to J5vgnd1, J11 to Jgnd12, J8 to Jpuerta1, Q3 to Qbuz1, Q1 to Qrelay1, Q2 to Qrele2, R9 to Rbot1, R10 to Rbot2, R14 to Rbuz1, R15 to Rldr1, R16 to Rldr2, R5 to Rled1, R6 to Rled2, R4 to Rled3, R3 to Rled4, R11 to Rpuerta1, R1 to Rrele1, R7 to Rrele12, R8 to Rrele2, R2 to Rrele2_1, R12 to Ru1, R13 to Ru2, R18 to Ruv2, R17 to Ruv21, SW3 to SWusb1, U3 to Uv2, J5 to bornrele2, J4 to borrele1
Routing:
- net +3.3V: track 37.6 -> 203.7 mm
- net GND: track 212.1 -> 359.8 mm
- net +5V: track 33.8 -> 152.6 mm
- net 5V PREVIO AL SWITCH: track 15.1 -> 110.7 mm
- net Net-(Drele12-A): track 15.3 -> 98.9 mm
- net Net-(D6-K): track 0.00 -> 49.4 mm
- net BOT_B: track 40.5 -> 6.36 mm
- net Net-(Drele1-A): track 6.12 -> 39.2 mm
- net BUZZER: track 0.00 -> 32.7 mm
- net PUERTA: track 4.96 -> 35.2 mm
- net Net-(borrele1-Pin_1): track 0.00 -> 28.7 mm
- net Net-(borrele1-Pin_2): track 0.00 -> 27.8 mm
- net LED-B2: track 12.2 -> 36.6 mm
- net Net-(bornrele2-Pin_2): track 0.00 -> 24.3 mm
- net Net-(borrele1-Pin_3): track 0.00 -> 19.5 mm
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
Commit message: si
Parts:
- D1, D2, D3, D4: footprint LED_THT:LED_D5.0mm -> Connector_Molex:Molex_KK-254_AE-6410-02A_1x02_P2.54mm_Vertical
- moved Dusb1 130.7 mm to (120.3, 68.5), turned to 0 degrees
- moved J10 106.2 mm to (133.0, 73.0), turned to 0 degrees
- moved J7 103.3 mm to (128.1, 79.8), turned to 180 degrees
- moved SWusb1 101.7 mm to (121.0, 90.9), turned to 0 degrees
- moved J9 95.5 mm to (133.0, 80.5), turned to 0 degrees
- moved J2 88.4 mm to (143.2, 68.5)
- moved J6 84.5 mm to (133.5, 88.0), turned to 0 degrees
- moved J3 82.8 mm to (131.5, 95.0), turned to 0 degrees
- moved Rbot1 74.5 mm to (121.4, 135.0)
- moved SW1 71.4 mm to (132.5, 131.0)
- moved Rldr1 46.3 mm to (167.6, 147.8)
- moved Rpuerta1 46.3 mm to (178.5, 160.0)
- moved Rldr2 46.3 mm to (179.5, 154.4)
- moved Jpuerta1 44.9 mm to (164.0, 154.5)
- moved D2 39.1 mm to (192.5, 76.5)
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Connections:
- J10 pad 1: GND -> +5V
- J10 pad 2: +5V -> GND
- U1 pad 11: RELE_B -> unconnected-(U1-IO35-Pad11)
- U1 pad 12: RELE_A -> unconnected-(U1-IO34-Pad12)
- U1 pad 13: unconnected-(U1-IO39-Pad13) -> BUZZER
- U1 pad 14: unconnected-(U1-IO36-Pad14) -> PUERTA
- U1 pad 18: LED-A1 -> unconnected-(U1-IO1-Pad18)
- U1 pad 22: unconnected-(U1-IO18-Pad22) -> RELE_A
- U1 pad 23: BUZZER -> RELE_B
- U1 pad 24: unconnected-(U1-IO17-Pad24) -> LED-A1
- U1 pad 25: unconnected-(U1-IO16-Pad25) -> LED-B2
- U1 pad 26: LED-B2 -> LED-B1
- U1 pad 27: LED-B1 -> LED-A2
- U1 pad 28: LED-A2 -> BOT_B
- U1 pad 8: PUERTA -> unconnected-(U1-IO25-Pad8)
- U1 pad 9: BOT_B -> unconnected-(U1-IO33-Pad9)
Routing:
- net GND: track 359.8 -> 97.4 mm
- net +3.3V: track 203.7 -> 41.5 mm
- net +5V: track 152.6 -> 34.1 mm
- net Net-(Drele12-A): track 98.9 -> 0.00 mm
- net 5V PREVIO AL SWITCH: track 110.7 -> 26.3 mm
- net Net-(D6-K): track 49.4 -> 0.00 mm
- net Net-(Drele1-A): track 39.2 -> 0.00 mm
- net LED-B2: track 36.6 -> 0.00 mm
- net SDA: track 8.76 -> 44.6 mm
- net PUERTA: track 35.2 -> 0.00 mm
- net +3V3: track 33.5 -> 0.00 mm
- net BUZZER: track 32.7 -> 0.00 mm
- net LED-B1: track 29.2 -> 0.00 mm
- net Net-(borrele1-Pin_1): track 28.7 -> 0.00 mm
- net Net-(borrele1-Pin_2): track 27.8 -> 0.00 mm
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
Commit message: aa
Parts:
- J2, J3: footprint Connector_Molex:Molex_KK-254_AE-6410-04A_1x04_P2.54mm_Vertical -> Connector_PinHeader_2.54mm:PinHeader_1x01_P2.54mm_Vertical
- moved Rldr2 130.2 mm to (56.5, 111.5), turned to 180 degrees
- moved Rldr1 129.6 mm to (41.5, 118.0)
- moved Qbuz1 114.3 mm to (32.0, 99.7), turned to -90 degrees
- moved SW1 108.9 mm to (35.3, 82.0), turned to 180 degrees
- moved Ru2 107.3 mm to (51.6, 122.5), turned to 180 degrees
- moved J3 106.1 mm to (30.5, 62.5)
- moved J5vgnd1 103.2 mm to (64.0, 145.4)
- moved Qrele2 102.5 mm to (164.7, 34.9)
- moved U2 101.5 mm to (50.5, 127.0)
- moved K2 101.2 mm to (169.6, 47.5)
- moved bornrele2 101.2 mm to (145.5, 53.1)
- moved Rrele2 100.9 mm to (150.9, 37.5)
- moved Ruv2 100.7 mm to (44.0, 146.9), turned to -90 degrees
- moved Ru1 100.0 mm to (46.6, 127.5)
- moved Cuv21 99.6 mm to (38.1, 147.9), turned to 90 degrees
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Connections:
- U1 pad 14: PUERTA -> unconnected-(U1-IO36-Pad14)
- U1 pad 21: unconnected-(U1-IO19-Pad21) -> BOT_B
- U1 pad 28: BOT_B -> unconnected-(U1-IO15-Pad28)
- U1 pad 7: unconnected-(U1-IO26-Pad7) -> PUERTA
Routing:
- net GND: track 97.4 -> 423.6 mm
- net +3.3V: track 41.5 -> 343.1 mm
- net +5V: track 34.1 -> 300.2 mm
- net 5V PREVIO AL SWITCH: track 26.3 -> 209.4 mm
- net RELE_A: track 0.00 -> 116.5 mm
- net LDR: track 0.00 -> 104.6 mm
- net PUERTA: track 0.00 -> 89.8 mm
- net Net-(Drele12-A): track 0.00 -> 86.4 mm
- net BOT_B: track 0.00 -> 59.2 mm, vias 0 -> 1
- net RELE_B: track 0.00 -> 54.4 mm
- net BUZZER: track 0.00 -> 40.2 mm, vias 0 -> 1
- net BOT_A: track 6.28 -> 42.7 mm, vias 0 -> 1
- net Net-(Drele1-A): track 0.00 -> 34.4 mm
- net +12V: track 0.00 -> 29.3 mm
- net Net-(bornrele2-Pin_2): track 0.00 -> 24.3 mm
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
Commit message: terminado
Parts:
- moved Jpuerta1 64.7 mm to (42.2, 91.0)
- moved Qrelay1 58.4 mm to (115.0, 87.5), turned to 0 degrees
- moved Ruv21 57.2 mm to (62.0, 113.9), turned to -90 degrees
- moved Drele1 55.7 mm to (109.9, 95.0), turned to 0 degrees
- moved Rpuerta1 55.1 mm to (58.0, 90.0)
- moved Qrele2 55.0 mm to (130.0, 77.5), turned to 90 degrees
- moved Rrele2_1 54.5 mm to (114.9, 67.5), turned to 0 degrees
- moved Rrele2 52.0 mm to (114.9, 75.0)
- moved Rrele1 50.1 mm to (127.5, 102.6), turned to 90 degrees
- moved K2 48.1 mm to (122.5, 57.5), turned to 90 degrees
- moved J5vgnd1 46.7 mm to (78.5, 101.0)
- moved borrele1 45.4 mm to (120.1, 122.5)
- moved K1 44.8 mm to (115.0, 99.5)
- moved Cu3 43.2 mm to (68.0, 101.9), turned to -90 degrees
- moved Rrele12 41.0 mm to (112.4, 80.0)
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Connections:
- U1 pad 16: BOT_A -> unconnected-(U1-IO23-Pad16)
- U1 pad 19: unconnected-(U1-IO3-Pad19) -> BOT_A
- U1 pad 22: RELE_A -> unconnected-(U1-IO18-Pad22)
- U1 pad 28: unconnected-(U1-IO15-Pad28) -> RELE_A
Routing:
- net +5V: track 300.2 -> 113.7 mm
- net +3.3V: track 343.1 -> 224.5 mm
- net RELE_A: track 116.5 -> 23.6 mm
- net LDR: track 104.6 -> 44.4 mm, vias 0 -> 4
- net Net-(Drele12-A): track 86.4 -> 31.4 mm
- net PUERTA: track 89.8 -> 56.0 mm, vias 0 -> 4
- net 5V PREVIO AL SWITCH: track 209.4 -> 176.7 mm, vias 0 -> 2
- net GND: track 423.6 -> 400.7 mm
- net RELE_B: track 54.4 -> 35.9 mm
- net Net-(D5-K): track 21.9 -> 7.44 mm
- net Net-(BZ1--): track 17.8 -> 4.70 mm
- net Net-(Drele1-A): track 34.4 -> 22.1 mm
- net +12V: track 29.3 -> 18.1 mm
- net LED-A2: track 23.3 -> 13.2 mm
- net Net-(Uv2-ADJ): track 21.8 -> 31.9 mm
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
Commit message: suuuuuu
Parts:
- moved Ru2 0.90 mm to (64.1, 97.2)
Connections:
- U1 pad 19: BOT_A -> unconnected-(U1-IO3-Pad19)
- U1 pad 22: unconnected-(U1-IO18-Pad22) -> BOT_A
Routing:
- net GND: track 400.7 -> 322.6 mm
- net 5V PREVIO AL SWITCH: track 176.7 -> 162.2 mm, vias 2 -> 0
- net BOT_A: track 38.7 -> 46.8 mm, vias 0 -> 2
- net PUERTA: track 56.0 -> 49.8 mm, vias 4 -> 2
- net +5V: track 113.7 -> 118.9 mm
- net LDR: track 44.4 -> 41.0 mm, vias 4 -> 0
- net BUZZER: track 31.6 -> 33.5 mm, vias 2 -> 0
- net +3.3V: track 224.5 -> 223.0 mm
- net LED-A1: track 14.7 -> 16.0 mm
- net Net-(D3-K): track 4.99 -> 3.97 mm
- net +3V3: track 21.9 -> 21.3 mm
- added copper zone on B.Cu, net GND
